File: Eagle/AxisNT_RF_PA.sch (EAGLE design)
At the start: 64 parts, among them IC1 74HCT259N, IC2 74HCT244N, IC3 74ALS08N, IC4 74ALS04N, U1 AD5308ARUZ, U10 LMV824MT, U2 AD5308ARUZ, U22 AD7994-0, U4 AD7994-0, U5 SC18IS602BIPW,112, U6 LMV824MT, U7 LMV824MT, U8 LMV824MT, U9 LM75A, U99 LMV824MT

Commit message: Add files via upload
Parts:
- removed IC1: 74HCT259N, 74xx-eu:74HCT259N
- removed IC2: 74HCT244N, 74xx-eu:74HCT244N
- removed REG1: (no value), v-reg:78LXX
- removed U$1: 25LC040/SN, Microchip_By_element14_Batch_1:25LC040/SN
- removed U5: SC18IS602BIPW,112, NXP_By_element14_Batch_1:SC18IS602BIPW,112
- added R1, R3, R30, R330: 10k, rcl:R-EU_R0402
- added R114, R118, R207, R211, R212, R315, R39: 100, rcl:R-EU_R0402
- added R150, R198, R?5: 10K, rcl:R-EU_R0402
- added R?3, R?4: 4.7K, rcl:R-EU_R0402
- added REG12: (no value), v-reg:78LXX
- added TP118, TP126: TPB1,27, testpad:TPB1,27
- added U12: 74HCT244N, 74xx-eu:74HCT244N
- added U14: 74HCT259N, 74xx-eu:74HCT259N
- added U19: 25LC040/SN, Microchip_By_element14_Batch_1:25LC040/SN
- added U26: SC18IS602BIPW,112, NXP_By_element14_Batch_1:SC18IS602BIPW,112
Connections:
- removed net N$1: IC4D.O, IC4E.I
- new net !EEPROM_CS: U14A.Q1, U19.~CS
- new net !HCT_LE: PL5.7, R114.1, TP118.TP
- new net !SYNC1: U14A.Q2, U2.~SYNC
- new net !SYNC2: U1.~SYNC, U14A.Q3
- new net !WP: U14A.Q7, U19.~WP
- new net HCT_D: PL4.7, R39.1, TP126.TP
- new net MISO: U19.SO, U26.MISO
- new net MOSI: U1.DIN, U12B.Y1, U19.SI, U2.DIN
- new net N$23: R211.1, U26.~SS0/GPIO0
- new net N$24: R211.2, U14A.S0
- new net N$25: R212.2, U14A.S1
- new net N$26: R212.1, U26.~SS1/GPIO1
- new net N$27: R207.2, U14A.S2
- new net N$28: R207.1, U26.~SS2/GPIO2
- new net N$29: R114.2, R330.2, U14A.G
- new net N$30: R3.1, U14A.CLR
- new net N$31: R30.2, R39.2, U14A.D
- new net N$32: R150.2, U26.~RESET
- new net N$33: R1.1, U19.~HOLD
- new net N$34: R118.2, U12A.A4
- new net N$35: R118.1, U26.SPICLK
- new net N$36: R?5.2, U2.~LDAC
- new net N$37: R198.2, U1.~LDAC
- new net N$38: R315.2, U12B.A1
- new net N$39: R315.1, U26.MOSI
- new net SCK: U1.SCLK, U12A.Y4, U19.SCK, U2.SCLK
- net !ADC_CONVST: now also U12A.Y3; no longer IC2A.Y3
- net +7V: now also REG12.IN; no longer REG1.IN
- net GND: now also R198.1, R30.1, R330.1, R?5.1, REG12.GND, U1.GND, U14P.GND, U19.VSS, U2.GND, U26.VSS; no longer REG1.GND, U5.VSS
- net N$16: now also U12A.G; no longer IC2A.G
- net N$19: now also U12B.G; no longer IC2B.G
- net N$20: now also U26.A0; no longer U5.A0
- net N$21: now also U26.A1; no longer U5.A1
- net N$22: now also U26.A2; no longer U5.A2
- net SCL: now also R?3.1, U26.SCL; no longer U5.SCL
- net SDA: now also R?4.1, U26.SDA; no longer U5.SDA
- net VCC1: now also R1.2, R3.2, R?3.2, R?4.2, REG12.OUT, U1.VDD, U14P.VCC, U19.VCC, U2.VDD; no longer REG1.OUT
- net VCC2: now also R150.1, U26.VDD; no longer U5.VDD
Other:
- moved on the sheet: C110, C37, C80, IC3A, IC3B, IC3C, IC3D, IC4A, IC4B, IC4C, IC4D, IC4E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

Commit message: Add files via upload
Parts:
- removed IC4: 74ALS04N, 74xx-eu:74ALS04N
- added R101, R34, R53, R60\, R61: 10K, rcl:R-EU_R0402
- added R248: 10k, rcl:R-EU_R0402
- added R47, R91: 100, rcl:R-EU_R0402
- added TP114, TP117, TP122, TP70, TP71, TP77, TP80: TPB1,27, testpad:TPB1,27
- added U18: 74ALS04N, 74xx-eu:74ALS04N
- R1: value 10k -> 100
Connections:
- new net !AD_CONV: PL5.6, R47.1, TP117.TP
- new net N$1: R1.2, R34.1, U12A.A1
- new net N$40: R61.1, U12B.A4
- new net N$41: R101.1, R91.2, U12A.A2
- new net N$42: TP70.TP, U12A.Y1, U18B.I
- new net N$43: TP71.TP, U12A.Y2, U18A.I
- new net N$44: R47.2, R53.1, U12A.A3
- new net N$45: R60\.1, U12B.A3
- new net N?6: U12B.Y2
- new net TX_EN1: PL4.3, R1.1, TP122.TP
- new net TX_EN2: PL5.3, R91.1, TP114.TP
- net !EEPROM_CS: now also TP80.TP
- net !WP: now also TP77.TP
- net GND: now also R101.2, R34.2, R53.2, R60\.2, R61.2, U12P.GND
- net MISO: now also U12B.A2
- net N$33: now also R248.1; no longer R1.1
- net VCC1: now also R248.2, U12P.VCC; no longer R1.2
Other:
- moved on the sheet: R1, R118, R155, R198, R243, R?5, REG10, TP118, TP126, TP72, U1, U19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

Commit message: Add files via upload
Parts:
- removed IC3: 74ALS08N, 74xx-eu:74ALS08N
- added R2, R5: 10k, rcl:R-EU_R0402
- added R4, R6: 100, rcl:R-EU_R0402
- added TP115, TP116, TP123: TPB1,27, testpad:TPB1,27
- added U13: 74ALS08N, 74xx-eu:74ALS08N
Connections:
- new net N$46: U13A.I1, U18A.O
- new net N$47: U13A.I0, U18B.O
- new net N$48: U13B.O, U18C.I
- new net N$49: U13A.O, U13B.I1, U13C.I0
- new net N$50: R2.2, R4.2, U13B.I0
- new net N$51: R5.2, R6.2, U13C.I1
- new net N$53: U13C.O, U18D.I
- new net N$?7: PL4.4, TP123.TP
- new net N?7: R4.1
- new net N?8: PL5.4, R6.1, TP115.TP
- new net N?9: PL5.5, TP116.TP
- net !AD_CONV: now also PL3.3
- net GND: now also R2.1, R5.1, U13P.GND, U18P.GND
- net VCC1: now also U13P.VCC, U18P.VCC
Other:
- moved on the sheet: PL4, PL5, R?3, R?4, TP113, TP114, TP117, TP118, TP122, TP126, U18C, U18D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

Commit message: Add files via upload
Parts:
- added R153: 10k, rcl:R-EU_R0402
- added TP119, TP28: TPB1,27, testpad:TPB1,27
- renumbered R2 to R55, R4 to R29, R5 to R331, R6 to R?6
Connections:
- removed net N$53: U13C.O, U18D.I
- removed net N$?7: PL4.4, TP123.TP
- new net N$52: R153.2, U18F.I
- new net TR26?: TP28.TP, U13C.O, U18D.I
- net GND: now also R153.1, TP119.TP
- net N?7: now also PL4.4, TP123.TP
Other:
- moved on the sheet: U18D, U18F
Changed lines of the file:
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@@
 <part name="GND38" library="supply1" deviceset="GND" device=""/>
 <part name="GND39" library="supply1" deviceset="GND" device=""/>
-<part name="R2" library="rcl" deviceset="R-EU_" device="R0402" value="10k"/>
+<part name="R55" library="rcl" deviceset="R-EU_" device="R0402" value="10k"/>
 <part name="GND40" library="supply1" deviceset="GND" device=""/>
-<part name="R4" library="rcl" deviceset="R-EU_" device="R0402" value="100"/>
+<part name="R29" library="rcl" deviceset="R-EU_" device="R0402" value="100"/>
 <part name="TP123" library="testpad" deviceset="TP" device="B1,27"/>
-<part name="R5" library="rcl" deviceset="R-EU_" device="R0402" value="10k"/>
+<part name="R331" library="rcl" deviceset="R-EU_" device="R0402" value="10k"/>
 <part name="GND41" library="supply1" deviceset="GND" device=""/>
-<part name="R6" library="rcl" deviceset="R-EU_" device="R0402" value="100"/>
+<part name="R?6" library="rcl" deviceset="R-EU_" device="R0402" value="100"/>
 <part name="TP115" library="testpad" deviceset="TP" device="B1,27"/>
 <part name="TP116" library="testpad" deviceset="TP" device="B1,27"/>
+<part name="TP119" library="testpad" deviceset="TP" device="B1,27"/>
+<part name="TP28" library="testpad" deviceset="TP" device="B1,27"/>
+<part name="R153" library="rcl" deviceset="R-EU_" device="R0402" value="10k"/>
+<part name="GND42" library="supply1" deviceset="GND" device=""/>
 </parts>
 <sheets>
@@
 <instance part="U18" gate="B" x="429.26" y="256.54"/>
 <instance part="U18" gate="C" x="508" y="251.46"/>
-<instance part="U18" gate="D" x="510.54" y="205.74"/>
+<instance part="U18" gate="D" x="518.16" y="205.74"/>
 <instance part="U18" gate="E" x="558.8" y="223.52"/>
-<instance part="U18" gate="F" x="561.34" y="208.28"/>
+<instance part="U18" gate="F" x="500.38" y="177.8"/>
 <instance part="U9" gate="G$1" x="73.66" y="175.26"/>
 <instance part="U1" gate="A" x="299.72" y="88.9"/>
@@
 <instance part="U13" gate="P" x="467.36" y="276.86" rot="R90"/>
 <instance part="GND39" gate="1" x="477.52" y="271.78"/>
-<instance part="R2" gate="G$1" x="464.82" y="220.98" rot="R90"/>
+<instance part="R55" gate="G$1" x="464.82" y="220.98" rot="R90"/>
 <instance part="GND40" gate="1" x="464.82" y="210.82"/>
-<instance part="R4" gate="G$1" x="457.2" y="231.14"/>
+<instance part="R29" gate="G$1" x="457.2" y="231.14"/>
 <instance part="TP123" gate="G$1" x="43.18" y="142.24"/>
-<instance part="R5" gate="G$1" x="464.82" y="193.04" rot="R90"/>
+<instance part="R331" gate="G$1" x="464.82" y="193.04" rot="R90"/>
 <instance part="GND41" gate="1" x="464.82" y="182.88"/>
-<instance part="R6" gate="G$1" x="457.2" y="203.2"/>
+<instance part="R?6" gate="G$1" x="457.2" y="203.2"/>
 <instance part="TP115" gate="G$1" x="63.5" y="266.7"/>
 <instance part="TP116" gate="G$1" x="76.2" y="264.16"/>
+<instance part="TP119" gate="G$1" x="33.02" y="187.96"/>
+<instance part="TP28" gate="G$1" x="505.46" y="213.36"/>
+<instance part="R153" gate="G$1" x="487.68" y="170.18" rot="R90"/>
+<instance part="GND42" gate="1" x="487.68" y="160.02"/>
 </instances>
 <busses>
@@
 <wire x1="20.32" y1="182.88" x2="25.4" y2="182.88" width="0.1524" layer="91"/>
 <wire x1="25.4" y1="182.88" x2="25.4" y2="180.34" width="0.1524" layer="91"/>
+<pinref part="TP119" gate="G$1" pin="TP"/>
+<wire x1="25.4" y1="182.88" x2="33.02" y2="182.88" width="0.1524" layer="91"/>
+<wire x1="33.02" y1="182.88" x2="33.02" y2="185.42" width="0.1524" layer="91"/>
+<junction x="25.4" y="182.88"/>
 </segment>
 <segment>
@@
 </segment>
 <segment>
-<pinref part="R2" gate="G$1" pin="1"/>
+<pinref part="R55" gate="G$1" pin="1"/>
 <pinref part="GND40" gate="1" pin="GND"/>
 <wire x1="464.82" y1="213.36" x2="464.82" y2="215.9" width="0.1524" layer="91"/>
 </segment>
 <segment>
-<pinref part="R5" gate="G$1" pin="1"/>
+<pinref part="R331" gate="G$1" pin="1"/>
 <pinref part="GND41" gate="1" pin="GND"/>
 <wire x1="464.82" y1="185.42" x2="464.82" y2="187.96" width="0.1524" layer="91"/>
+</segment>
+<segment>
+<pinref part="R153" gate="G$1" pin="1"/>
+<pinref part="GND42" gate="1" pin="GND"/>
+<wire x1="487.68" y1="162.56" x2="487.68" y2="165.1" width="0.1524" layer="91"/>
 </segment>
 </net>
@@
 <net name="N$50" class="0">
 <segment>
-<pinref part="R2" gate="G$1" pin="2"/>
+<pinref part="R55" gate="G$1" pin="2"/>
 <wire x1="474.98" y1="231.14" x2="464.82" y2="231.14" width="0.1524" layer="91"/>
 <wire x1="464.82" y1="231.14" x2="464.82" y2="226.06" width="0.1524" layer="91"/>
-<pinref part="R4" gate="G$1" pin="2"/>
+<pinref part="R29" gate="G$1" pin="2"/>
 <wire x1="462.28" y1="231.14" x2="464.82" y2="231.14" width="0.1524" layer="91"/>
 <junction x="464.82" y="231.14"/>
@@
 <net name="N?7" class="0">
 <segment>
-<pinref part="R4" gate="G$1" pin="1"/>
+<pinref part="R29" gate="G$1" pin="1"/>
 <wire x1="452.12" y1="231.14" x2="449.58" y2="231.14" width="0.1524" layer="91"/>
 <label x="449.58" y="231.14" size="1.778" layer="95" rot="R180" xref="yes"/>
 </segment>
-</net>
-<net name="N$?7" class="0">
 <segment>
 <pinref part="PL4" gate="A" pin="4"/>
@@
 <net name="N$51" class="0">
 <segment>
-<pinref part="R5" gate="G$1" pin="2"/>
+<pinref part="R331" gate="G$1" pin="2"/>
 <wire x1="482.6" y1="203.2" x2="464.82" y2="203.2" width="0.1524" layer="91"/>
 <wire x1="464.82" y1="203.2" x2="464.82" y2="198.12" width="0.1524" layer="91"/>
-<pinref part="R6" gate="G$1" pin="2"/>
+<pinref part="R?6" gate="G$1" pin="2"/>
 <wire x1="462.28" y1="203.2" x2="464.82" y2="203.2" width="0.1524" layer="91"/>
 <junction x="464.82" y="203.2"/>
@@
 <net name="N?8" class="0">
 <segment>
-<pinref part="R6" gate="G$1" pin="1"/>
+<pinref part="R?6" gate="G$1" pin="1"/>
 <wire x1="452.12" y1="203.2" x2="449.58" y2="203.2" width="0.1524" layer="91"/>
 <label x="449.58" y="203.2" size="1.778" layer="95" rot="R180" xref="yes"/>
@@
 </segment>
 </net>
-<net name="N$53" class="0">
+<net name="TR26?" class="0">
 <segment>
 <pinref part="U13" gate="C" pin="O"/>
 <pinref part="U18" gate="D" pin="I"/>
-<wire x1="500.38" y1="205.74" x2="497.84" y2="205.74" width="0.1524" layer="91"/>
-</segment>
-</net>
+<wire x1="508" y1="205.74" x2="505.46" y2="205.74" width="0.1524" layer="91"/>
+<pinref part="TP28" gate="G$1" pin="TP"/>
+<wire x1="505.46" y1="205.74" x2="497.84" y2="205.74" width="0.1524" layer="91"/>
+<wire x1="505.46" y1="210.82" x2="505.46" y2="205.74" width="0.1524" layer="91"/>
+<junction x="505.46" y="205.74"/>
+<wire x1="505.46" y1="205.74" x2="505.46" y2="190.5" width="0.1524" layer="91"/>
+<wire x1="505.46" y1="190.5" x2="508" y2="190.5" width="0.1524" layer="91"/>
+<label x="508" y="190.5" size="1.778" layer="95" xref="yes"/>
+</segment>
+</net>
+<net name="N$52" class="0">
+<segment>
+<pinref part="U18" gate="F" pin="I"/>
+<pinref part="R153" gate="G$1" pin="2"/>
+<wire x1="490.22" y1="177.8" x2="487.68" y2="177.8" width="0.1524" layer="91"/>
+<wire x1="487.68" y1="177.8" x2="487.68" y2="175.26" width="0.1524" layer="91"/>
+</segment>
+</net>
