File: Eagle/AxisNT_RF_PA.sch (EAGLE design)
At the start: 107 parts, among them U1 AD5308ARUZ, U10 LMV824MT, U12 74HCT244N, U13 74ALS08N, U14 74HCT259N, U18 74ALS04N, U19 25LC040/SN, U2 AD5308ARUZ, U22 AD7994-0, U26 SC18IS602BIPW,112, U4 AD7994-0, U6 LMV824MT, U7 LMV824MT, U8 LMV824MT, U9 LM75A, U99 LMV824MT

Commit message: VCC voltage update
Connections:
- net VCC1 renamed +5V
- new net +3V3: REG10.OUT, TP15.TP, U26.VDD
- net VCC2: no longer REG10.OUT, TP15.TP, U26.VDD
