File: Eagle/AxisNT_RF_PA.sch (EAGLE design)
At the start: 107 parts, among them U1 AD5308ARUZ, U10 LMV824MT, U12 74HCT244N, U13 74ALS08N, U14 74HCT259N, U18 74ALS04N, U19 25LC040/SN, U2 AD5308ARUZ, U22 AD7994-0, U26 SC18IS602BIPW,112, U4 AD7994-0, U6 LMV824MT, U7 LMV824MT, U8 LMV824MT, U9 LM75A, U99 LMV824MT

Commit message: Add files via upload
Parts:
- added TP105, TP108, TP2, TP75, TP76, TP85, TP86, TP87, TP88, TP97, TP98, TP?2: TPB1,27, testpad:TPB1,27
Connections:
- new net APM1_TR14_TP51: TP85.TP
- new net N$53: TP105.TP, U1.VOUTB
- new net N$54: TP2.TP, U1.VOUTG
- new net N$55: TP86.TP, U2.VOUTB
- new net N$56: TP98.TP, U1.VOUTA
- new net N$57: TP?2.TP, U2.VOUTE
- new net N$58: U2.VOUTF
- new net N$59: U2.VOUTG
- new net N$60: TP75.TP, U14A.Q0, U18E.I
- new net N$61: TP76.TP, U18E.O
- net APM1_TR11_TP84_TP111: now also TP87.TP
- net APM1_TR12_TP83_TP48: now also TP88.TP
- net APM2_TR28_TP108_TP32: now also TP108.TP
- net APM2_TR3_TP96_TP112: now also TP97.TP
Other:
- moved on the sheet: U18E
Changed lines of the file:
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@@
 <part name="GND42" library="supply1" deviceset="GND" device=""/>
 <part name="+3V1" library="supply1" deviceset="+3V3" device=""/>
+<part name="TP87" library="testpad" deviceset="TP" device="B1,27"/>
+<part name="TP88" library="testpad" deviceset="TP" device="B1,27"/>
+<part name="TP97" library="testpad" deviceset="TP" device="B1,27"/>
+<part name="TP108" library="testpad" deviceset="TP" device="B1,27"/>
+<part name="TP105" library="testpad" deviceset="TP" device="B1,27"/>
+<part name="TP2" library="testpad" deviceset="TP" device="B1,27"/>
+<part name="TP85" library="testpad" deviceset="TP" device="B1,27"/>
+<part name="TP86" library="testpad" deviceset="TP" device="B1,27"/>
+<part name="TP98" library="testpad" deviceset="TP" device="B1,27"/>
+<part name="TP?2" library="testpad" deviceset="TP" device="B1,27"/>
+<part name="TP75" library="testpad" deviceset="TP" device="B1,27"/>
+<part name="TP76" library="testpad" deviceset="TP" device="B1,27"/>
 </parts>
 <sheets>
@@
 <instance part="U18" gate="C" x="508" y="251.46"/>
 <instance part="U18" gate="D" x="518.16" y="205.74"/>
-<instance part="U18" gate="E" x="558.8" y="223.52"/>
+<instance part="U18" gate="E" x="436.88" y="182.88"/>
 <instance part="U18" gate="F" x="500.38" y="177.8"/>
 <instance part="U9" gate="G$1" x="73.66" y="175.26"/>
@@
 <instance part="GND42" gate="1" x="487.68" y="160.02"/>
 <instance part="+3V1" gate="G$1" x="289.56" y="193.04"/>
+<instance part="TP87" gate="G$1" x="337.82" y="50.8"/>
+<instance part="TP88" gate="G$1" x="332.74" y="45.72"/>
+<instance part="TP97" gate="G$1" x="340.36" y="106.68"/>
+<instance part="TP108" gate="G$1" x="332.74" y="101.6"/>
+<instance part="TP105" gate="G$1" x="327.66" y="106.68"/>
+<instance part="TP2" gate="G$1" x="325.12" y="68.58" rot="R180"/>
+<instance part="TP85" gate="G$1" x="325.12" y="53.34"/>
+<instance part="TP86" gate="G$1" x="327.66" y="50.8"/>
+<instance part="TP98" gate="G$1" x="325.12" y="101.6"/>
+<instance part="TP?2" gate="G$1" x="325.12" y="17.78" rot="R180"/>
+<instance part="TP75" gate="G$1" x="424.18" y="190.5"/>
+<instance part="TP76" gate="G$1" x="449.58" y="190.5"/>
 </instances>
 <busses>
@@
 <segment>
 <pinref part="U1" gate="A" pin="VOUTD"/>
-<wire x1="322.58" y1="88.9" x2="325.12" y2="88.9" width="0.1524" layer="91"/>
-<label x="325.12" y="88.9" size="1.778" layer="95" xref="yes"/>
+<wire x1="322.58" y1="88.9" x2="340.36" y2="88.9" width="0.1524" layer="91"/>
+<label x="342.9" y="88.9" size="1.778" layer="95" xref="yes"/>
+<pinref part="TP97" gate="G$1" pin="TP"/>
+<wire x1="340.36" y1="88.9" x2="342.9" y2="88.9" width="0.1524" layer="91"/>
+<wire x1="340.36" y1="104.14" x2="340.36" y2="88.9" width="0.1524" layer="91"/>
+<junction x="340.36" y="88.9"/>
 </segment>
 </net>
@@
 <segment>
 <pinref part="U1" gate="A" pin="VOUTC"/>
-<wire x1="322.58" y1="91.44" x2="325.12" y2="91.44" width="0.1524" layer="91"/>
-<label x="325.12" y="91.44" size="1.778" layer="95" xref="yes"/>
+<wire x1="322.58" y1="91.44" x2="332.74" y2="91.44" width="0.1524" layer="91"/>
+<label x="342.9" y="91.44" size="1.778" layer="95" xref="yes"/>
+<pinref part="TP108" gate="G$1" pin="TP"/>
+<wire x1="332.74" y1="91.44" x2="342.9" y2="91.44" width="0.1524" layer="91"/>
+<wire x1="332.74" y1="99.06" x2="332.74" y2="91.44" width="0.1524" layer="91"/>
+<junction x="332.74" y="91.44"/>
 </segment>
 </net>
@@
 <segment>
 <pinref part="U2" gate="A" pin="VOUTD"/>
-<wire x1="322.58" y1="38.1" x2="325.12" y2="38.1" width="0.1524" layer="91"/>
-<label x="325.12" y="38.1" size="1.778" layer="95" xref="yes"/>
+<wire x1="322.58" y1="38.1" x2="337.82" y2="38.1" width="0.1524" layer="91"/>
+<label x="342.9" y="38.1" size="1.778" layer="95" xref="yes"/>
+<pinref part="TP87" gate="G$1" pin="TP"/>
+<wire x1="337.82" y1="38.1" x2="342.9" y2="38.1" width="0.1524" layer="91"/>
+<wire x1="337.82" y1="48.26" x2="337.82" y2="38.1" width="0.1524" layer="91"/>
+<junction x="337.82" y="38.1"/>
 </segment>
 </net>
@@
 <segment>
 <pinref part="U2" gate="A" pin="VOUTC"/>
-<wire x1="322.58" y1="40.64" x2="325.12" y2="40.64" width="0.1524" layer="91"/>
-<label x="325.12" y="40.64" size="1.778" layer="95" xref="yes"/>
-</segment>
-</net>
+<wire x1="322.58" y1="40.64" x2="332.74" y2="40.64" width="0.1524" layer="91"/>
+<label x="342.9" y="40.64" size="1.778" layer="95" xref="yes"/>
+<pinref part="TP88" gate="G$1" pin="TP"/>
+<wire x1="332.74" y1="40.64" x2="342.9" y2="40.64" width="0.1524" layer="91"/>
+<wire x1="332.74" y1="43.18" x2="332.74" y2="40.64" width="0.1524" layer="91"/>
+<junction x="332.74" y="40.64"/>
+</segment>
+</net>
+<net name="N$53" class="0">
+<segment>
+<pinref part="U1" gate="A" pin="VOUTB"/>
+<pinref part="TP105" gate="G$1" pin="TP"/>
+<wire x1="322.58" y1="93.98" x2="327.66" y2="93.98" width="0.1524" layer="91"/>
+<wire x1="327.66" y1="93.98" x2="327.66" y2="104.14" width="0.1524" layer="91"/>
+<junction x="327.66" y="93.98"/>
+<wire x1="327.66" y1="93.98" x2="342.9" y2="93.98" width="0.1524" layer="91"/>
+<label x="342.9" y="93.98" size="1.778" layer="95" xref="yes"/>
+</segment>
+</net>
+<net name="N$54" class="0">
+<segment>
+<pinref part="U1" gate="A" pin="VOUTG"/>
+<pinref part="TP2" gate="G$1" pin="TP"/>
+<wire x1="322.58" y1="81.28" x2="325.12" y2="81.28" width="0.1524" layer="91"/>
+<wire x1="325.12" y1="81.28" x2="325.12" y2="71.12" width="0.1524" layer="91"/>
+<wire x1="325.12" y1="81.28" x2="342.9" y2="81.28" width="0.1524" layer="91"/>
+<junction x="325.12" y="81.28"/>
+<label x="342.9" y="81.28" size="1.778" layer="95" xref="yes"/>
+</segment>
+</net>
+<net name="APM1_TR14_TP51" class="0">
+<segment>
+<pinref part="TP85" gate="G$1" pin="TP"/>
+<wire x1="320.04" y1="45.72" x2="325.12" y2="45.72" width="0.1524" layer="91"/>
+<wire x1="325.12" y1="45.72" x2="325.12" y2="50.8" width="0.1524" layer="91"/>
+<wire x1="325.12" y1="45.72" x2="342.9" y2="45.72" width="0.1524" layer="91"/>
+<junction x="325.12" y="45.72"/>
+<label x="342.9" y="45.72" size="1.778" layer="95" xref="yes"/>
+</segment>
+</net>
+<net name="N$55" class="0">
+<segment>
+<pinref part="U2" gate="A" pin="VOUTB"/>
+<pinref part="TP86" gate="G$1" pin="TP"/>
+<wire x1="322.58" y1="43.18" x2="327.66" y2="43.18" width="0.1524" layer="91"/>
+<wire x1="327.66" y1="43.18" x2="327.66" y2="48.26" width="0.1524" layer="91"/>
+<wire x1="327.66" y1="43.18" x2="342.9" y2="43.18" width="0.1524" layer="91"/>
+<junction x="327.66" y="43.18"/>
+<label x="342.9" y="43.18" size="1.778" layer="95" xref="yes"/>
+</segment>
+</net>
+<net name="N$56" class="0">
+<segment>
+<pinref part="U1" gate="A" pin="VOUTA"/>
+<pinref part="TP98" gate="G$1" pin="TP"/>
+<wire x1="322.58" y1="96.52" x2="325.12" y2="96.52" width="0.1524" layer="91"/>
+<wire x1="325.12" y1="96.52" x2="325.12" y2="99.06" width="0.1524" layer="91"/>
+<wire x1="325.12" y1="96.52" x2="342.9" y2="96.52" width="0.1524" layer="91"/>
+<junction x="325.12" y="96.52"/>
+<label x="342.9" y="96.52" size="1.778" layer="95" xref="yes"/>
+</segment>
+</net>
+<net name="N$57" class="0">
+<segment>
+<pinref part="U2" gate="A" pin="VOUTE"/>
+<wire x1="322.58" y1="35.56" x2="325.12" y2="35.56" width="0.1524" layer="91"/>
+<wire x1="325.12" y1="35.56" x2="325.12" y2="20.32" width="0.1524" layer="91"/>
+<pinref part="TP?2" gate="G$1" pin="TP"/>
+<wire x1="325.12" y1="35.56" x2="342.9" y2="35.56" width="0.1524" layer="91"/>
+<junction x="325.12" y="35.56"/>
+<label x="342.9" y="35.56" size="1.778" layer="95" xref="yes"/>
+</segment>
+</net>
+<net name="N$58" class="0">
+<segment>
+<pinref part="U2" gate="A" pin="VOUTF"/>
+<wire x1="322.58" y1="33.02" x2="342.9" y2="33.02" width="0.1524" layer="91"/>
+<label x="342.9" y="33.02" size="1.778" layer="95" xref="yes"/>
+</segment>
+</net>
+<net name="N$59" class="0">
+<segment>
+<pinref part="U2" gate="A" pin="VOUTG"/>
+<wire x1="322.58" y1="30.48" x2="342.9" y2="30.48" width="0.1524" layer="91"/>
+<label x="342.9" y="30.48" size="1.778" layer="95" xref="yes"/>
+</segment>
+</net>
+<net name="N$60" class="0">
+<segment>
+<pinref part="U14" gate="A" pin="Q0"/>
+<wire x1="421.64" y1="167.64" x2="424.18" y2="167.64" width="0.1524" layer="91"/>
+<wire x1="424.18" y1="167.64" x2="424.18" y2="182.88" width="0.1524" layer="91"/>
+<pinref part="U18" gate="E" pin="I"/>
+<wire x1="424.18" y1="182.88" x2="426.72" y2="182.88" width="0.1524" layer="91"/>
+<pinref part="TP75" gate="G$1" pin="TP"/>
+<wire x1="424.18" y1="182.88" x2="424.18" y2="187.96" width="0.1524" layer="91"/>
+<junction x="424.18" y="182.88"/>
+</segment>
+</net>
+<net name="N$61" class="0">
+<segment>
+<pinref part="U18" gate="E" pin="O"/>
+<wire x1="447.04" y1="182.88" x2="449.58" y2="182.88" width="0.1524" layer="91"/>
+<wire x1="449.58" y1="182.88" x2="449.58" y2="187.96" width="0.1524" layer="91"/>
+<pinref part="TP76" gate="G$1" pin="TP"/>
+</segment>
+</net>

Commit message: Add Gambas3 Project
Parts:
- added TP121: TPB1,27, testpad:TPB1,27
Connections:
- net N?7 renamed RX_EN1
- net N?8 renamed RX_EN2
- new net MISO??: PL4.2, TP121.TP
- new net TO_RX1: U18C.O
- new net TO_RX2: U18D.O
Other:
- moved on the sheet: TP116, TP122, TP123, TP126
Changed lines of the file:
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@@
 <part name="TP75" library="testpad" deviceset="TP" device="B1,27"/>
 <part name="TP76" library="testpad" deviceset="TP" device="B1,27"/>
+<part name="TP121" library="testpad" deviceset="TP" device="B1,27"/>
 </parts>
 <sheets>
@@
 <instance part="GND26" gate="1" x="381" y="167.64"/>
 <instance part="R39" gate="G$1" x="373.38" y="187.96"/>
-<instance part="TP126" gate="G$1" x="58.42" y="137.16"/>
+<instance part="TP126" gate="G$1" x="63.5" y="137.16"/>
 <instance part="R150" gate="G$1" x="269.24" y="167.64"/>
 <instance part="R?3" gate="G$1" x="38.1" y="274.32" rot="R90"/>
@@
 <instance part="GND31" gate="1" x="274.32" y="17.78"/>
 <instance part="R315" gate="G$1" x="320.04" y="205.74" rot="R90"/>
-<instance part="TP122" gate="G$1" x="27.94" y="144.78"/>
+<instance part="TP122" gate="G$1" x="30.48" y="147.32"/>
 <instance part="R1" gate="G$1" x="294.64" y="256.54"/>
 <instance part="R34" gate="G$1" x="332.74" y="236.22" rot="R270"/>
@@
 <instance part="GND40" gate="1" x="464.82" y="210.82"/>
 <instance part="R29" gate="G$1" x="457.2" y="231.14"/>
-<instance part="TP123" gate="G$1" x="43.18" y="142.24"/>
+<instance part="TP123" gate="G$1" x="45.72" y="142.24"/>
 <instance part="R331" gate="G$1" x="464.82" y="193.04" rot="R90"/>
 <instance part="GND41" gate="1" x="464.82" y="182.88"/>
 <instance part="R?6" gate="G$1" x="457.2" y="203.2"/>
 <instance part="TP115" gate="G$1" x="63.5" y="266.7"/>
-<instance part="TP116" gate="G$1" x="76.2" y="264.16"/>
+<instance part="TP116" gate="G$1" x="78.74" y="264.16"/>
 <instance part="TP119" gate="G$1" x="33.02" y="187.96"/>
 <instance part="TP28" gate="G$1" x="505.46" y="213.36"/>
@@
 <instance part="TP75" gate="G$1" x="424.18" y="190.5"/>
 <instance part="TP76" gate="G$1" x="449.58" y="190.5"/>
+<instance part="TP121" gate="G$1" x="27.94" y="149.86"/>
 </instances>
 <busses>
@@
 <pinref part="PL4" gate="A" pin="7"/>
 <pinref part="TP126" gate="G$1" pin="TP"/>
-<wire x1="20.32" y1="129.54" x2="58.42" y2="129.54" width="0.1524" layer="91"/>
-<wire x1="58.42" y1="129.54" x2="58.42" y2="134.62" width="0.1524" layer="91"/>
-<wire x1="58.42" y1="129.54" x2="60.96" y2="129.54" width="0.1524" layer="91"/>
-<junction x="58.42" y="129.54"/>
-<label x="60.96" y="129.54" size="1.778" layer="95" xref="yes"/>
+<wire x1="20.32" y1="129.54" x2="63.5" y2="129.54" width="0.1524" layer="91"/>
+<wire x1="63.5" y1="129.54" x2="63.5" y2="134.62" width="0.1524" layer="91"/>
+<wire x1="63.5" y1="129.54" x2="66.04" y2="129.54" width="0.1524" layer="91"/>
+<junction x="63.5" y="129.54"/>
+<label x="66.04" y="129.54" size="1.778" layer="95" xref="yes"/>
 </segment>
 </net>
@@
 <segment>
 <pinref part="PL4" gate="A" pin="3"/>
-<wire x1="20.32" y1="139.7" x2="27.94" y2="139.7" width="0.1524" layer="91"/>
+<wire x1="20.32" y1="139.7" x2="30.48" y2="139.7" width="0.1524" layer="91"/>
 <pinref part="TP122" gate="G$1" pin="TP"/>
-<wire x1="27.94" y1="139.7" x2="30.48" y2="139.7" width="0.1524" layer="91"/>
-<wire x1="27.94" y1="142.24" x2="27.94" y2="139.7" width="0.1524" layer="91"/>
-<junction x="27.94" y="139.7"/>
-<label x="30.48" y="139.7" size="1.778" layer="95" xref="yes"/>
+<wire x1="30.48" y1="139.7" x2="33.02" y2="139.7" width="0.1524" layer="91"/>
+<wire x1="30.48" y1="144.78" x2="30.48" y2="139.7" width="0.1524" layer="91"/>
+<junction x="30.48" y="139.7"/>
+<label x="33.02" y="139.7" size="1.778" layer="95" xref="yes"/>
 </segment>
 <segment>
@@
 </segment>
 </net>
-<net name="N?7" class="0">
+<net name="RX_EN1" class="0">
 <segment>
 <pinref part="R29" gate="G$1" pin="1"/>
@@
 <segment>
 <pinref part="PL4" gate="A" pin="4"/>
-<wire x1="20.32" y1="137.16" x2="43.18" y2="137.16" width="0.1524" layer="91"/>
+<wire x1="20.32" y1="137.16" x2="45.72" y2="137.16" width="0.1524" layer="91"/>
 <pinref part="TP123" gate="G$1" pin="TP"/>
-<wire x1="43.18" y1="137.16" x2="45.72" y2="137.16" width="0.1524" layer="91"/>
-<wire x1="43.18" y1="139.7" x2="43.18" y2="137.16" width="0.1524" layer="91"/>
-<junction x="43.18" y="137.16"/>
-<label x="45.72" y="137.16" size="1.778" layer="95" xref="yes"/>
+<wire x1="45.72" y1="137.16" x2="48.26" y2="137.16" width="0.1524" layer="91"/>
+<wire x1="45.72" y1="139.7" x2="45.72" y2="137.16" width="0.1524" layer="91"/>
+<junction x="45.72" y="137.16"/>
+<label x="48.26" y="137.16" size="1.778" layer="95" xref="yes"/>
 </segment>
 </net>
@@
 </segment>
 </net>
-<net name="N?8" class="0">
+<net name="RX_EN2" class="0">
 <segment>
 <pinref part="R?6" gate="G$1" pin="1"/>
@@
 <segment>
 <pinref part="PL5" gate="A" pin="5"/>
-<wire x1="22.86" y1="256.54" x2="76.2" y2="256.54" width="0.1524" layer="91"/>
+<wire x1="22.86" y1="256.54" x2="78.74" y2="256.54" width="0.1524" layer="91"/>
 <pinref part="TP116" gate="G$1" pin="TP"/>
-<wire x1="76.2" y1="256.54" x2="78.74" y2="256.54" width="0.1524" layer="91"/>
-<wire x1="76.2" y1="261.62" x2="76.2" y2="256.54" width="0.1524" layer="91"/>
-<junction x="76.2" y="256.54"/>
-<label x="78.74" y="256.54" size="1.778" layer="95" xref="yes"/>
+<wire x1="78.74" y1="256.54" x2="81.28" y2="256.54" width="0.1524" layer="91"/>
+<wire x1="78.74" y1="261.62" x2="78.74" y2="256.54" width="0.1524" layer="91"/>
+<junction x="78.74" y="256.54"/>
+<label x="81.28" y="256.54" size="1.778" layer="95" xref="yes"/>
 </segment>
 </net>
@@
 </segment>
 </net>
+<net name="TO_RX1" class="0">
+<segment>
+<pinref part="U18" gate="C" pin="O"/>
+<wire x1="518.16" y1="251.46" x2="523.24" y2="251.46" width="0.1524" layer="91"/>
+<label x="523.24" y="251.46" size="1.778" layer="95" xref="yes"/>
+</segment>
+</net>
+<net name="TO_RX2" class="0">
+<segment>
+<pinref part="U18" gate="D" pin="O"/>
+<wire x1="528.32" y1="205.74" x2="530.86" y2="205.74" width="0.1524" layer="91"/>
+<label x="530.86" y="205.74" size="1.778" layer="95" xref="yes"/>
+</segment>
+</net>
+<net name="MISO??" class="0">
+<segment>
+<pinref part="PL4" gate="A" pin="2"/>
+<wire x1="20.32" y1="142.24" x2="27.94" y2="142.24" width="0.1524" layer="91"/>
+<wire x1="27.94" y1="142.24" x2="43.18" y2="142.24" width="0.1524" layer="91"/>
+<wire x1="43.18" y1="142.24" x2="43.18" y2="147.32" width="0.1524" layer="91"/>
+<wire x1="43.18" y1="147.32" x2="55.88" y2="147.32" width="0.1524" layer="91"/>
+<label x="55.88" y="147.32" size="1.778" layer="95" xref="yes"/>
+<pinref part="TP121" gate="G$1" pin="TP"/>
+<wire x1="27.94" y1="142.24" x2="27.94" y2="147.32" width="0.1524" layer="91"/>
+<junction x="27.94" y="142.24"/>
+</segment>
+</net>
